File: KiCAD Files/LED PCB/PCB.kicad_pcb (KiCad board)
At the start: 2 copper layers, 66 x 55.9 mm, 52 parts, among them J1 Conn_01x18_Male, J2 Conn_01x18_Male, SW1 SW_Push, SW2 SW_Push, SW3 SW_Push, SW4 SW_Push, SW5 SW_Push, SW6 SW_Push, SW7 SW_Push

Commit message: Updated schematic. Added tooloing hole for driver for potential assembly. Added rev number
Routing:
- net /R6: track 90.3 -> 93.6 mm
Other:
- board text added: "Rev 1.0"
Changed lines of the file:
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@@
   (gr_arc (start 185.42 53.34) (end 185.42 50.8) (angle -90) (layer "Edge.Cuts") (width 0.1))
   (gr_line (start 182.88 53.34) (end 182.88 104.14) (layer "Edge.Cuts") (width 0.1))
+  (gr_text "Rev 1.0\n" (at 242.316 61.976) (layer "B.SilkS")
+    (effects (font (size 1.5 1.5) (thickness 0.2032)) (justify left mirror))
+  )
   (gr_text "4-In-A-Row Soldering Kit LED Board" (at 242.57 56.515) (layer "B.SilkS")
     (effects (font (size 1.5 1.5) (thickness 0.2032)) (justify left mirror))
@@
   (segment (start 243.84 82.55) (end 242.824 83.566) (width 0.381) (layer "B.Cu") (net 5))
   (segment (start 246.38 82.55) (end 243.84 82.55) (width 0.381) (layer "B.Cu") (net 5))
-  (segment (start 197.993 105.664) (end 200.025 103.632) (width 0.381) (layer "F.Cu") (net 6))
-  (segment (start 220.853 105.664) (end 228.473 105.664) (width 0.381) (layer "F.Cu") (net 6))
+  (segment (start 235.585 105.156) (end 236.093 105.664) (width 0.381) (layer "F.Cu") (net 6))
   (segment (start 236.093 105.664) (end 238.125 103.632) (width 0.381) (layer "F.Cu") (net 6))
-  (segment (start 213.233 105.664) (end 215.265 103.632) (width 0.381) (layer "F.Cu") (net 6))
-  (segment (start 197.993 105.664) (end 205.613 105.664) (width 0.381) (layer "F.Cu") (net 6))
-  (segment (start 205.613 105.664) (end 207.645 103.632) (width 0.381) (layer "F.Cu") (net 6))
-  (segment (start 228.473 105.664) (end 230.505 103.632) (width 0.381) (layer "F.Cu") (net 6))
-  (segment (start 228.473 105.664) (end 236.093 105.664) (width 0.381) (layer "F.Cu") (net 6))
-  (segment (start 194.437 105.664) (end 197.993 105.664) (width 0.381) (layer "F.Cu") (net 6))
-  (segment (start 205.613 105.664) (end 213.233 105.664) (width 0.381) (layer "F.Cu") (net 6))
-  (segment (start 213.233 105.664) (end 220.853 105.664) (width 0.381) (layer "F.Cu") (net 6))
-  (segment (start 192.405 103.632) (end 194.437 105.664) (width 0.381) (layer "F.Cu") (net 6))
-  (segment (start 220.853 105.664) (end 222.885 103.632) (width 0.381) (layer "F.Cu") (net 6))
+  (segment (start 212.344 105.156) (end 213.741 105.156) (width 0.381) (layer "F.Cu") (net 6))
+  (segment (start 196.85 105.156) (end 198.501 105.156) (width 0.381) (layer "F.Cu") (net 6))
+  (segment (start 192.405 103.632) (end 193.929 105.156) (width 0.381) (layer "F.Cu") (net 6))
+  (segment (start 193.929 105.156) (end 198.501 105.156) (width 0.381) (layer "F.Cu") (net 6))
+  (segment (start 213.741 105.156) (end 215.265 103.632) (width 0.381) (layer "F.Cu") (net 6))
+  (segment (start 204.851 105.156) (end 206.121 105.156) (width 0.381) (layer "F.Cu") (net 6))
+  (segment (start 198.501 105.156) (end 200.025 103.632) (width 0.381) (layer "F.Cu") (net 6))
+  (segment (start 221.361 105.156) (end 222.885 103.632) (width 0.381) (layer "F.Cu") (net 6))
+  (segment (start 227.711 105.156) (end 235.585 105.156) (width 0.381) (layer "F.Cu") (net 6))
+  (segment (start 220.091 105.156) (end 228.981 105.156) (width 0.381) (layer "F.Cu") (net 6))
+  (segment (start 206.121 105.156) (end 207.645 103.632) (width 0.381) (layer "F.Cu") (net 6))
+  (segment (start 198.501 105.156) (end 206.121 105.156) (width 0.381) (layer "F.Cu") (net 6))
+  (segment (start 228.981 105.156) (end 230.505 103.632) (width 0.381) (layer "F.Cu") (net 6))
+  (segment (start 206.121 105.156) (end 213.741 105.156) (width 0.381) (layer "F.Cu") (net 6))
+  (segment (start 213.741 105.156) (end 221.361 105.156) (width 0.381) (layer "F.Cu") (net 6))
   (via (at 236.093 105.664) (size 0.8128) (drill 0.3302) (layers "F.Cu" "B.Cu") (net 6))
   (segment (start 244.348 87.122) (end 244.348 103.759) (width 0.381) (layer "B.Cu") (net 6))
@@
   (segment (start 225.933 92.202) (end 225.933 92.329) (width 0.381) (layer "B.Cu") (net 27))
   (segment (start 225.933 103.632) (end 225.933 92.329) (width 0.381) (layer "B.Cu") (net 27))
-  (segment (start 185.42 54.229) (end 188.214 51.435) (width 0.381) (layer "F.Cu") (net 28))
-  (segment (start 234.918 51.435) (end 236.673 53.19) (width 0.381) (layer "F.Cu") (net 28))
-  (segment (start 188.214 51.435) (end 234.918 51.435) (width 0.381) (layer "F.Cu") (net 28))
-  (segment (start 185.42 57.15) (end 185.42 54.229) (width 0.381) (layer "F.Cu") (net 28))
+  (segment (start 185.42 54.229) (end 187.96 51.689) (width 0.254) (layer "F.Cu") (net 28))
+  (segment (start 185.42 57.15) (end 185.42 54.229) (width 0.254) (layer "F.Cu") (net 28))
+  (segment (start 235.172 51.689) (end 236.673 53.19) (width 0.254) (layer "F.Cu") (net 28))
+  (segment (start 187.96 51.689) (end 235.172 51.689) (width 0.254) (layer "F.Cu") (net 28))
   (segment (start 236.8 53.317) (end 236.673 53.19) (width 0.381) (layer "B.Cu") (net 28))
   (segment (start 236.8 59.563) (end 236.8 53.317) (width 0.381) (layer "B.Cu") (net 28))
